File: 01-led/01-led.kicad_pcb (KiCad board)
At the start: 2 copper layers, 12.7 x 16.5 mm, 4 parts, among them J1 Conn_01x02_Socket, J2 Conn_01x02_Socket

Commit message: add image
Routing:
- added copper zone on F.Cu, net GND
Changed lines of the file:
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@@
     (pad "2" thru_hole circle (at 2.54 0 90) (size 1.8 1.8) (drill 0.9) (layers "*.Cu" "*.Mask")
       (net 2 "Net-(D1-A)") (pinfunction "A") (pintype "passive"))
-    (model "${KICAD6_3DMODEL_DIR}/LED_THT.3dshapes/LED_D3.0mm.wrl"
-      (offset (xyz 0 0 -3.175))
+    (model "/home/obijuan/Develop/Learn-Kicad/3D/LEDS/LED_D3-2.0mm.step"
+      (offset (xyz 1.27 0 0))
       (scale (xyz 1 1 1))
       (rotate (xyz 0 0 0))
@@
       (net 3 "Net-(D2-A)") (pinfunction "A") (pintype "passive"))
     (model "${KICAD6_3DMODEL_DIR}/LED_THT.3dshapes/LED_D3.0mm.wrl"
-      (offset (xyz 0 0 -3.175))
+      (offset (xyz 0 0 0))
       (scale (xyz 1 1 1))
       (rotate (xyz 0 0 0))
@@
   (segment (start 138.938 86.868) (end 137.16 85.09) (width 0.381) (layer "F.Cu") (net 3))
   (segment (start 134.62 96.52) (end 137.668 96.52) (width 0.381) (layer "F.Cu") (net 3))
+  (zone (net 1) (net_name "GND") (layer "F.Cu") (hatch edge 0.5)
+    (connect_pads (clearance 0.5))
+    (min_thickness 0.25) (filled_areas_thickness no)
+    (fill yes (thermal_gap 0.5) (thermal_bridge_width 0.5))
+    (polygon
+      (pts
+        (xy 128.524 82.804)
+        (xy 140.716 82.804)
+        (xy 140.716 98.806)
+        (xy 128.524 98.806)
+      )
+    )
+  )
 )
